Commit message: Entorno y correcion de paquetes

File: urdf/bcr_bot.xacro (robot description, xacro)
@@ -1,4 +1,4 @@
 <?xml version="1.0"?>
-<robot xmlns:xacro="http://www.ros.org/wiki/xacro" name="bcr_bot">
+<robot xmlns:xacro="http://www.ros.org/wiki/xacro" name="carga_bot">
     <!--................................ XACRO CONSTANTS .............................. -->
     <xacro:property name="chassis_mass" value="70"/>
@@ -42,14 +42,14 @@
     <xacro:property name="odometry_source" value="$(arg odometry_source)"/>
     <!-- ............................... LOAD MACROS ................................. -->
-    <xacro:include filename="$(find bcr_bot)/urdf/materials.xacro"/>
-    <xacro:include filename="$(find bcr_bot)/urdf/macros.xacro"/>
+    <xacro:include filename="$(find carga_bot)/urdf/materials.xacro"/>
+    <xacro:include filename="$(find carga_bot)/urdf/macros.xacro"/>
     <xacro:if value="$(arg sim_gazebo)">
-        <xacro:include filename="$(find bcr_bot)/urdf/gazebo.xacro"/>
+        <xacro:include filename="$(find carga_bot)/urdf/gazebo.xacro"/>
     </xacro:if>
     <xacro:if value="$(arg sim_ign)">
-        <xacro:include filename="$(find bcr_bot)/urdf/ign.xacro"/>
+        <xacro:include filename="$(find carga_bot)/urdf/ign.xacro"/>
     </xacro:if>
     <xacro:if value="$(arg sim_gz)">
-        <xacro:include filename="$(find bcr_bot)/urdf/gz.xacro"/>
+        <xacro:include filename="$(find carga_bot)/urdf/gz.xacro"/>
     </xacro:if>
     <!-- ................................ BASE LINK .................................. -->
@@ -71,5 +71,5 @@
             <origin xyz="0 0 -0.205" rpy="0 0 0" />
             <geometry>
-                <mesh filename="file://$(find bcr_bot)/meshes/bcr_bot_mesh.dae" scale="1 1 1"/>
+                <mesh filename="file://$(find carga_bot)/meshes/carga_bot_mesh.dae" scale="1 1 1"/>
             </geometry>
         </visual>
@@ -142,5 +142,5 @@
                 <origin xyz="0 0 0" rpy="0 0 0" />
                 <geometry>
-                    <mesh filename="file://$(find bcr_bot)/meshes/kinect/d415.dae"/>
+                    <mesh filename="file://$(find carga_bot)/meshes/kinect/d415.dae"/>
                 </geometry>
                 <material name="black"/>
@@ -176,5 +176,5 @@
                 <origin xyz="0 0 0" rpy="0 0 0" />
                 <geometry>
-                    <mesh filename="file://$(find bcr_bot)/meshes/kinect/d415.dae"/>
+                    <mesh filename="file://$(find carga_bot)/meshes/kinect/d415.dae"/>
                 </geometry>
                 <material name="black"/>

File: urdf/gazebo.xacro (robot description, xacro)
@@ -1,4 +1,4 @@
 <?xml version="1.0"?>
-<robot xmlns:xacro="http://www.ros.org/wiki/xacro" name="bcr_bot">
+<robot xmlns:xacro="http://www.ros.org/wiki/xacro" name="carga_bot">
     <gazebo>
         <static>false</static>

File: urdf/gz.xacro (robot description, xacro)
@@ -1,4 +1,4 @@
 <?xml version="1.0"?>
-<robot xmlns:xacro="http://www.ros.org/wiki/xacro" name="bcr_bot">
+<robot xmlns:xacro="http://www.ros.org/wiki/xacro" name="carga_bot">
     <!-- ........................... SENSOR PLUGIN ................................... -->
     <gazebo>

File: urdf/ign.xacro (robot description, xacro)
@@ -1,4 +1,4 @@
 <?xml version="1.0"?>
-<robot xmlns:xacro="http://www.ros.org/wiki/xacro" name="bcr_bot">
+<robot xmlns:xacro="http://www.ros.org/wiki/xacro" name="carga_bot">
     <!-- ........................... SENSOR PLUGIN ................................... -->
     <gazebo>

File: urdf/macros.xacro (robot description, xacro)
@@ -1,4 +1,4 @@
 <?xml version="1.0"?>
-<robot xmlns:xacro="http://www.ros.org/wiki/xacro" name="bcr_bot">
+<robot xmlns:xacro="http://www.ros.org/wiki/xacro" name="carga_bot">
     <!--................................ INERTIA MATRICES .............................. -->
     <xacro:macro name="cylinder_inertia" params="m r h">

File: urdf/materials.xacro (robot description, xacro)
@@ -1,4 +1,4 @@
 <?xml version="1.0"?>
-<robot xmlns:xacro="http://www.ros.org/wiki/xacro" name="bcr_bot">
+<robot xmlns:xacro="http://www.ros.org/wiki/xacro" name="carga_bot">
     <material name="black">
         <color rgba="0.0 0.0 0.0 1.0"/>
