Commit message: agregar la carga y redisenio de bot

File: urdf/carga_bot.xacro (robot description, xacro)
@@ -215,4 +215,23 @@
         <origin xyz="0 0 0.16" rpy="0 0 0" />
     </joint>
+    <!-- ............................. CARGA ........................................ -->
+    <link name= "carga_link">
+        <visual>
+                <origin xyz="0 0 0" rpy="0 0 0" />
+                <geometry>
+                    <box size= "${chassis_length} ${chassis_width} 0.9"/>
+                </geometry>
+                <material name="carton"/>
+        </visual>
+        <inertial>
+            <mass value="1"/>
+            <xacro:box_inertia m="50" x="1" y="0.6" z = "0.9"/>
+        </inertial>
+    </link>
+    <joint name="carga_joint" type="fixed">
+        <parent link="chassis_link"/>
+        <child link="carga_link"/>
+        <origin xyz="0 0 ${chassis_height/2+0.49}" rpy="0 0 0.0" />
+    </joint>
     <!-- ............................. CONVEYOR ........................................ -->
     <xacro:if value="$(arg conveyor_enabled)">

File: urdf/materials.xacro (robot description, xacro)
@@ -40,3 +40,6 @@
         <color rgba="0.1 0.1 0.1 1"/>
     </material>
+    <material name="carton">
+        <color rgba="0.76 0.60 0.42 1.0"/>
+    </material>
 </robot>
